Commit message: 2017/10/01 gazebo

File: catkin_ws/src/duckiebot-simulator/mybot/mybot_description/urdf/mybot.xacro (robot description, xacro)
@@ -3,12 +3,13 @@
   <xacro:property name="cameraSize" value="0.05"/>
   <xacro:property name="cameraMass" value="0.1"/>
+  <xacro:arg name="veh" default="$(arg veh)"/>
   <xacro:include filename="$(find mybot_description)/urdf/mybot.gazebo" />
-  <xacro:include filename="$(find mybot_description)/urdf/materials.xacro" />
-  <xacro:include filename="$(find mybot_description)/urdf/macros.xacro" />
+  <!--xacro:include filename="$(find mybot_description)/urdf/materials.xacro" /-->
+  <!--xacro:include filename="$(find mybot_description)/urdf/macros.xacro" /-->
   <link name='chassis'>
     <pose>0 0 0.1 0 0 0</pose>
     <inertial>
       <mass value="15.0"/>
-      <origin xyz="0.0 0 0.1" rpy=" 0 0 0"/>
+      <origin xyz="0.1 0 0.1" rpy=" 0 0 0"/>
       <inertia
           ixx="0.1" ixy="0" ixz="0"
