Commit message: apriltags following

File: catkin_ws/src/odometry/model/me212_robot.xacro (robot description, xacro)
@@ -4,5 +4,5 @@
     <visual>
         <geometry>
-            <mesh scale="0.001 0.001 0.001" filename="package://me212_robot/model/meshes/visual/me212_robot.stl"/>
+            <mesh scale="0.001 0.001 0.001" filename="package://odometry/model/meshes/visual/me212_robot.stl"/>
         </geometry>
         <material name="blue">
